File: SWD-UART-CTX-10.kicad_sch (KiCad schematic)
At the start: 16 parts, among them J1 UE25BE5510H, J2 3020-10-0100-00, J3 SFH11-PBPC-D10-RA-BK, J4 Pins_2.54_1x2, U1 USBLC6-2P6, U2 FT230XQ

Commit message: Just use headers
Parts:
- removed C1, C3: 100n, C_Capacitor:C_0603, symbol C_Capacitor:C_0603
- removed C2: 10u, C_Capacitor:C_0805, symbol C_Capacitor:C_0805
- removed DS1: LED_GRN, DS_LED:DS_0603, symbol DS_LED:DS_0603
- removed DS2: LED_YEL, DS_LED:DS_0603, symbol DS_LED:DS_0603
- removed J1: UE25BE5510H, J_Connector:USB_Mini_TH_Vertical, symbol J_Connector:UE25BE5510H
- removed L1: 600R, L_Inductor:FB_0603, symbol L_Inductor:FB_0603
- removed R1, R2, R3, R4: 470R, R_Resistor:R_0603, symbol R_Resistor:R_0603
- removed U1: USBLC6-2P6, U_IC:SOT23_6, symbol U_Basic:USBLC6-2P6
- removed U2: FT230XQ, U_IC:QFN16_065_4x4_EP, symbol U_Transceiver:FT230XQ
- added J1: 61300611121, J_Connector:Pins-2.54-1x6, symbol J_Connector:Pins_2.54_1x6
- J4: value Pins_2.54_1x2 -> 61300211121
Connections:
- net GND: now also J1.1
- net RXD: now also J1.5
- net TXD: now also J1.4
Other:
- note removed: "Detect"
- moved on the sheet: J2, J3, J4

Commit message: Add series R
Parts:
- added R1, R2: 470R, R_Resistor:R_0603, symbol R_Resistor:R_0603
Connections:
- net RXD: now also R1.1; no longer J1.5
- net TXD: now also R2.1; no longer J1.4
- new net: J1.4, R2.2
- new net: J1.5, R1.2
Changed lines of the file:
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@@
     (stroke (width 0) (type default) (color 0 0 0 0))
   )
-  (wire (pts (xy 104.14 73.66) (xy 106.68 73.66))
+  (wire (pts (xy 83.82 73.66) (xy 106.68 73.66))
     (stroke (width 0) (type default) (color 0 0 0 0))
   )
@@
     (stroke (width 0) (type default) (color 0 0 0 0))
   )
+  (wire (pts (xy 74.93 71.12) (xy 85.09 71.12))
+    (stroke (width 0) (type default) (color 0 0 0 0))
+  )
   (wire (pts (xy 176.53 78.74) (xy 176.53 74.93))
     (stroke (width 0) (type default) (color 0 0 0 0))
@@
     (stroke (width 0) (type default) (color 0 0 0 0))
   )
-  (wire (pts (xy 104.14 71.12) (xy 106.68 71.12))
+  (wire (pts (xy 90.17 71.12) (xy 106.68 71.12))
     (stroke (width 0) (type default) (color 0 0 0 0))
   )
@@
     (stroke (width 0) (type default) (color 0 0 0 0))
   )
+  (wire (pts (xy 74.93 73.66) (xy 78.74 73.66))
+    (stroke (width 0) (type default) (color 0 0 0 0))
+  )
   (wire (pts (xy 191.77 88.9) (xy 194.31 88.9))
     (stroke (width 0) (type default) (color 0 0 0 0))
@@
     (effects (font (size 1.27 1.27)) (justify left bottom))
   )
+  (label "TXD" (at 74.93 71.12 180)
+    (effects (font (size 1.27 1.27)) (justify right bottom))
+  )
   (label "VAUX" (at 139.7 91.44 180)
     (effects (font (size 1.27 1.27)) (justify right bottom))
@@
     (effects (font (size 1.27 1.27)) (justify left bottom))
   )
+  (label "RXD" (at 74.93 73.66 180)
+    (effects (font (size 1.27 1.27)) (justify right bottom))
+  )
   (label "SWCLK" (at 163.83 88.9 0)
     (effects (font (size 1.27 1.27)) (justify left bottom))
   )
-  (label "TXD" (at 104.14 71.12 180)
-    (effects (font (size 1.27 1.27)) (justify right bottom))
-  )
   (label "SWO" (at 163.83 91.44 0)
     (effects (font (size 1.27 1.27)) (justify left bottom))
-  )
-  (label "RXD" (at 104.14 73.66 180)
-    (effects (font (size 1.27 1.27)) (justify right bottom))
   )
   (label "SWDIO" (at 163.83 86.36 0)
@@
     (pin "1")
   )
+  (symbol (lib_id "R_Resistor:R_0603") (at 81.28 73.66 90) (unit 1)
+    (in_bom yes) (on_board yes) (fields_autoplaced)
+    (property "Reference" "R1" (id 0) (at 81.28 67.242 90))
+    (property "Value" "470R" (id 1) (at 81.28 69.7789 90))
+    (property "Footprint" "R_Resistor:R_0603" (id 2) (at 81.28 76.2 90)
+      (effects (font (size 1.27 1.27)) hide)
+    )
+    (property "Datasheet" "" (id 3) (at 85.09 76.2 0)
+      (effects (font (size 1.27 1.27)) hide)
+    )
+    (property "Size" "R_0603" (id 4) (at 81.28 71.7452 90)
+      (effects (font (size 0.635 0.635)))
+    )
+    (pin "1")
+    (pin "2")
+  )
   (symbol (lib_id "power:GND") (at 152.4 57.15 0) (unit 1)
     (in_bom yes) (on_board yes)
@@
     (property "Datasheet" "" (id 3) (at 146.05 50.8 0)
       (effects (font (size 1.27 1.27)) hide)
+    )
+    (pin "1")
+    (pin "2")
+  )
+  (symbol (lib_id "R_Resistor:R_0603") (at 87.63 71.12 90) (unit 1)
+    (in_bom yes) (on_board yes) (fields_autoplaced)
+    (property "Reference" "R2" (id 0) (at 87.63 64.702 90))
+    (property "Value" "470R" (id 1) (at 87.63 67.2389 90))
+    (property "Footprint" "R_Resistor:R_0603" (id 2) (at 87.63 73.66 90)
+      (effects (font (size 1.27 1.27)) hide)
+    )
+    (property "Datasheet" "" (id 3) (at 91.44 73.66 0)
+      (effects (font (size 1.27 1.27)) hide)
+    )
+    (property "Size" "R_0603" (id 4) (at 87.63 69.2052 90)
+      (effects (font (size 0.635 0.635)))
     )
     (pin "1")
@@
       (reference "J4") (unit 1) (value "61300211121") (footprint "J_Connector:Pins-2.54-1x2")
     )
-  )
+    (path "/7593b7eb-fb0e-41c5-b360-634f3beb25b9"
+      (reference "R1") (unit 1) (value "470R") (footprint "R_Resistor:R_0603")
+    )
+    (path "/a684abf6-bef7-4318-8458-99b3c02ccccd"
+      (reference "R2") (unit 1) (value "470R") (footprint "R_Resistor:R_0603")
+    )
+  )

Commit message: Add jumper for vaux to vbus
Parts:
- added JP1: SolderJumper_2_Open, Jumper:SolderJumper-2_P1.3mm_Open_Pad1.0x1.5mm, symbol Jumper:SolderJumper_2_Open
Connections:
- net VAUX: now also JP1.1 (A)
- net at J3.19 (Pin_19): now also JP1.2 (B)
Other:
- moved on the sheet: J4
Changed lines of the file:
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@@
   (junction (at 194.31 93.98) (diameter 0) (color 0 0 0 0)
   )
-  (wire (pts (xy 152.4 54.61) (xy 152.4 57.15))
+  (wire (pts (xy 148.59 123.19) (xy 148.59 125.73))
     (stroke (width 0) (type default) (color 0 0 0 0))
   )
@@
     (stroke (width 0) (type default) (color 0 0 0 0))
   )
-  (wire (pts (xy 149.86 54.61) (xy 152.4 54.61))
+  (wire (pts (xy 146.05 123.19) (xy 148.59 123.19))
     (stroke (width 0) (type default) (color 0 0 0 0))
   )
@@
     (stroke (width 0) (type default) (color 0 0 0 0))
   )
+  (wire (pts (xy 176.53 120.65) (xy 176.53 101.6))
+    (stroke (width 0) (type default) (color 0 0 0 0))
+  )
   (wire (pts (xy 154.94 86.36) (xy 179.07 86.36))
     (stroke (width 0) (type default) (color 0 0 0 0))
@@
     (stroke (width 0) (type default) (color 0 0 0 0))
   )
+  (wire (pts (xy 176.53 101.6) (xy 179.07 101.6))
+    (stroke (width 0) (type default) (color 0 0 0 0))
+  )
   (wire (pts (xy 194.31 99.06) (xy 194.31 96.52))
     (stroke (width 0) (type default) (color 0 0 0 0))
@@
     (stroke (width 0) (type default) (color 0 0 0 0))
   )
-  (wire (pts (xy 149.86 52.07) (xy 152.4 52.07))
-    (stroke (width 0) (type default) (color 0 0 0 0))
-  )
   (wire (pts (xy 154.94 88.9) (xy 179.07 88.9))
     (stroke (width 0) (type default) (color 0 0 0 0))
@@
     (stroke (width 0) (type default) (color 0 0 0 0))
   )
+  (wire (pts (xy 146.05 120.65) (xy 158.75 120.65))
+    (stroke (width 0) (type default) (color 0 0 0 0))
+  )
   (wire (pts (xy 90.17 71.12) (xy 106.68 71.12))
     (stroke (width 0) (type default) (color 0 0 0 0))
@@
   )
   (wire (pts (xy 101.6 63.5) (xy 106.68 63.5))
+    (stroke (width 0) (type default) (color 0 0 0 0))
+  )
+  (wire (pts (xy 166.37 120.65) (xy 176.53 120.65))
     (stroke (width 0) (type default) (color 0 0 0 0))
   )
@@
     (effects (font (size 1.27 1.27)) (justify left bottom))
   )
-  (label "VAUX" (at 152.4 52.07 0)
+  (label "VAUX" (at 148.59 120.65 0)
     (effects (font (size 1.27 1.27)) (justify left bottom))
   )
@@
     (pin "2")
   )
-  (symbol (lib_id "power:GND") (at 152.4 57.15 0) (unit 1)
-    (in_bom yes) (on_board yes)
-    (property "Reference" "#PWR013" (id 0) (at 152.4 63.5 0)
-      (effects (font (size 1.27 1.27)) hide)
-    )
-    (property "Value" "GND" (id 1) (at 152.4 64.77 90)
+  (symbol (lib_id "power:GND") (at 148.59 125.73 0) (unit 1)
+    (in_bom yes) (on_board yes)
+    (property "Reference" "#PWR013" (id 0) (at 148.59 132.08 0)
+      (effects (font (size 1.27 1.27)) hide)
+    )
+    (property "Value" "GND" (id 1) (at 148.59 133.35 90)
       (effects (font (size 1.27 1.27)) (justify left))
     )
-    (property "Footprint" "" (id 2) (at 152.4 57.15 0)
-      (effects (font (size 1.27 1.27)) hide)
-    )
-    (property "Datasheet" "" (id 3) (at 152.4 57.15 0)
-      (effects (font (size 1.27 1.27)) hide)
-    )
-    (pin "1")
-  )
-  (symbol (lib_id "J_Connector:Pins_2.54_1x2") (at 146.05 50.8 180) (unit 1)
-    (in_bom yes) (on_board yes) (fields_autoplaced)
-    (property "Reference" "J4" (id 0) (at 146.05 47.151 0))
-    (property "Value" "61300211121" (id 1) (at 146.05 49.6879 0))
-    (property "Footprint" "J_Connector:Pins-2.54-1x2" (id 2) (at 146.05 47.625 0)
-      (effects (font (size 1.27 1.27)) hide)
-    )
-    (property "Datasheet" "" (id 3) (at 146.05 50.8 0)
+    (property "Footprint" "" (id 2) (at 148.59 125.73 0)
+      (effects (font (size 1.27 1.27)) hide)
+    )
+    (property "Datasheet" "" (id 3) (at 148.59 125.73 0)
+      (effects (font (size 1.27 1.27)) hide)
+    )
+    (pin "1")
+  )
+  (symbol (lib_id "Jumper:SolderJumper_2_Open") (at 162.56 120.65 0) (unit 1)
+    (in_bom yes) (on_board yes)
+    (property "Reference" "JP1" (id 0) (at 163.83 118.11 0))
+    (property "Value" "SolderJumper_2_Open" (id 1) (at 163.83 123.19 0))
+    (property "Footprint" "Jumper:SolderJumper-2_P1.3mm_Open_Pad1.0x1.5mm" (id 2) (at 162.56 120.65 0)
+      (effects (font (size 1.27 1.27)) hide)
+    )
+    (property "Datasheet" "~" (id 3) (at 162.56 120.65 0)
+      (effects (font (size 1.27 1.27)) hide)
+    )
+    (pin "1")
+    (pin "2")
+  )
+  (symbol (lib_id "J_Connector:Pins_2.54_1x2") (at 142.24 119.38 180) (unit 1)
+    (in_bom yes) (on_board yes)
+    (property "Reference" "J4" (id 0) (at 142.24 115.731 0))
+    (property "Value" "61300211121" (id 1) (at 142.24 118.2679 0))
+    (property "Footprint" "J_Connector:Pins-2.54-1x2" (id 2) (at 142.24 116.205 0)
+      (effects (font (size 1.27 1.27)) hide)
+    )
+    (property "Datasheet" "" (id 3) (at 142.24 119.38 0)
       (effects (font (size 1.27 1.27)) hide)
     )
@@
       (reference "J4") (unit 1) (value "61300211121") (footprint "J_Connector:Pins-2.54-1x2")
     )
+    (path "/9bd596e6-ac94-439a-9562-6b698e3145cd"
+      (reference "JP1") (unit 1) (value "SolderJumper_2_Open") (footprint "Jumper:SolderJumper-2_P1.3mm_Open_Pad1.0x1.5mm")
+    )
     (path "/7593b7eb-fb0e-41c5-b360-634f3beb25b9"

Commit message: Update for J-Link options
Parts:
- removed J1: 61300611121, J_Connector:Pins-2.54-1x6, symbol J_Connector:Pins_2.54_1x6
- removed JP1: SolderJumper_2_Open, Jumper:SolderJumper-2_P1.3mm_Open_Pad1.0x1.5mm, symbol Jumper:SolderJumper_2_Open
- added J1: 61301221121, Connector_PinHeader_2.54mm:PinHeader_2x06_P2.54mm_Vertical, symbol Connector_Generic:Conn_02x06_Odd_Even
- J4: footprint J_Connector:Pins-2.54-1x2 -> Connector_PinHeader_2.54mm:PinHeader_1x02_P2.54mm_Vertical
Connections:
- net GND: now also J1.1 (Pin_1), J1.2 (Pin_2); no longer J4.1
- net VAUX: now also J4.1; no longer J4.2
- net at R2.2: now also J1.7 (Pin_7)
- net at R1.2: now also J1.9 (Pin_9)
- net VBUS_PROG: now reaches J3.19 (Pin_19)
- net VBUS_PROG: now also J1.6 (Pin_6)
- net RXD_PROG: now reaches J3.17 (Pin_17)
- net RXD_PROG: now also J1.10 (Pin_10)
- net TXD_PROG: now reaches J3.5 (Pin_5)
- net TXD_PROG: now also J1.8 (Pin_8)
- new net VBUS: J1.5 (Pin_5), J4.2
- no-connect marks 0 -> 6
Other:
- note added: "Connects VBUS to VAUX."
- note added: "Suggested jumper is: M7581-05"
- note added: "These pins can be used for a FTDI cable, or as jumpers to connect to a J-Link"
- note added: "To TC2050 / EC10 ribbon"
- note added: "To standard 20 pin programmer, such as JLink or STLink."
- moved on the sheet: J3
